File: pcb/LEDs.kicad_sch (KiCad schematic)
At the start: 66 parts, among them U76 74AHCT125

Commit message: feat: assigned footprints for each symbol and switch
Parts:
- R70: renamed from R4; footprint (none) -> Resistor_SMD:R_0603_1608Metric
- U76: footprint (none) -> prometheus-65-footprints:SN74AUC08RGYRG4
- renumbered D32 to D17, D31 to D18, D30 to D19, D29 to D20, D28 to D21, D27 to D22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
